File: src/L0005-Valve-Controller/L0005-Valve-Controller.sch (KiCad schematic (older format))
At the start: 60 parts, among them J1 Jumper_NO, J2 Jumper_NO, P1 3220-20-0200-00, P10 353620650, P11 353620650, P12 353620650, P13 353620650, P14 647676-3, P15 647676-3, P16 647676-2, P2 140-504-415-000, P9 647676-2, U1 LPC54113J256BD64QL, U2 LMS8117AMP-3.3_NOPB, U3 MAX3370EXK+T, U4 MAX3370EXK+T, U5 Optocoupler

Commit message: routed solenoid SSRs
Parts:
- B1: footprint SW_PTS647SM38SMTR2LFS_CNK -> L0005-Valve-Controller:PTS647SM38SMTR2LFS
- C1, C10, C11, C12, C13, C2, C22, C23, C24, C25, C3, C4, C5, C6, C7, C8, C9: footprint (none) -> L0005-Valve-Controller:CAP_0603
- C14, C15: footprint (none) -> Engine-Controller:CWR11HH106KB
- D1, D2: footprint (none) -> L0005-Valve-Controller:SML-LX1206GC-TR
- D3: footprint (none) -> L0005-Valve-Controller:150120AS75000
- D4: footprint (none) -> L0005-Valve-Controller:LED_RED
- F1: footprint FUSC9830X318N -> L0005-Valve-Controller:FUSC9830X318N
- J1, J2: footprint (none) -> L0005-Valve-Controller:Jumper-NO
- P1: footprint CONN20_D10-RA-BK_SUL -> L0005-Valve-Controller:3220-20-0200-00
- P10, P11, P12, P13: footprint CONN_4840.2201_SCH -> L0005-Valve-Controller:MOLEX_35362-0650
- P14, P15: footprint CONN_2043-1X04G00DAU_OUP -> L0005-Valve-Controller:647676-3
- P16, P9: footprint CONN_2043-1X04G00DAU_OUP -> L0005-Valve-Controller:TE_647676-2
- P2: footprint CONN_4840.2201_SCH -> L0005-Valve-Controller:140-504-415-000
- R1, R14, R15, R16, R17, R18, R19, R20, R21, R22, R23, R24, R25: footprint (none) -> L0005-Valve-Controller:RES_0603
- TP1, TP2, TP3, TP4, TP5: footprint (none) -> L0005-Valve-Controller:TP
- U1: footprint LQFP64_10X10_NXP -> L0005-Valve-Controller:LPC54113J256BD64QL
- U2: footprint (none) -> L0005-Valve-Controller:LMS8117AMP-3.3NOPB
- U3, U4: footprint 21-0076E_MXM -> L0005-Valve-Controller:MAX3370EXK&plus_T
- U5: footprint Package_DIP:DIP-4_W7.62mm -> L0005-Valve-Controller:Opto_140105146000
