File: src/L0005-Valve-Controller/L0005-Valve-Controller.kicad_pcb (KiCad board)
At the start: 4 copper layers, 141.7 x 50.5 mm, 102 parts, among them J1 Jumper_NO, J2 Jumper_NO, K1 AQH0223AX, K2 AQH0223AX, K3 AQH0223AX, K4 AQH0223AX, K5 AQH0223AX, K6 AQH0223AX, P1 3220-20-0200-00, P10 353620650, P11 353620650, P12 353620650, P13 353620650, P14 647676-3, P15 647676-3, P16 647676-2, P2 140-504-415-000, P3 647676-3, P4 647676-3, P5 647676-3, P6 647676-3, P7 647676-3, P8 647676-3, P9 647676-2, Q1 CMLDM7003, Q2 CMLDM7003, U1 LPC54113J256BD64QL, U2 LMS8117AMP-3.3_NOPB, U3 MAX3370EXK+T, U4 MAX3370EXK+T, U5 Optocoupler

Commit message: plotted schematic to pdf
Parts:
- removed H4: Mounting-Hole, L0005-Valve-Controller:MountingHole_4.3mm_M4_DIN965
- removed J2: Jumper_NO, L0005-Valve-Controller:Jumper-NO
- added H2: Mounting-Hole, L0005-Valve-Controller:MountingHole_4.3mm_M4_DIN965, F.Cu at (165.8, 58.6)
- added R26: 100k, L0005-Valve-Controller:RES_0603, F.Cu at (132.4, 74.3)
- added R27: 100k, L0005-Valve-Controller:RES_0603, F.Cu at (128.0, 76.5)
- B1: value SW_PTS647SM38SMTR2LFS_CNK -> PTS647SM38SMTR2LFS
- C1, C2: value 0.1uF -> 10uF; footprint L0005-Valve-Controller:CAP_0603 -> L0005-Valve-Controller:T491A106K010AT
- C11: value 0.1uF -> 2.2uF
- C12, C13: value 10nF -> 2.2uF
- C14: value 10uF -> 2.2uF; footprint L0005-Valve-Controller:T491A106K010AT -> L0005-Valve-Controller:CAP_0603
- C15: value 10uF -> 0.1uF; footprint L0005-Valve-Controller:T491A106K010AT -> L0005-Valve-Controller:CAP_0603
- C3: value 10uF -> 0.1uF
- C4, C5: value 10nF -> 0.1uF
- C8: value 0.1uF -> 4.7uF
- C9: value 10uF -> 1uF
- TP2, TP3, TP4, TP5: moved to F.Cu
- U1: value LPC54113J256BD64QL -> STM32H750VBTx; footprint L0005-Valve-Controller:LPC54113J256BD64QL -> L0005-Valve-Controller:STM32H750VBT6
- moved H1 102.9 mm to (149.5, 68.5)
- moved H3 97.3 mm to (158.6, 68.5)
- moved P16 91.3 mm to (129.3, 25.5)
- moved P9 87.2 mm to (139.3, 25.5)
- moved TP4 85.2 mm to (169.5, 27.6)
- moved C5 83.5 mm to (166.9, 25.0)
- moved R22 82.9 mm to (165.9, 30.8), turned to 0 degrees
- moved C6 82.0 mm to (166.0, 28.2)
- moved TP5 81.8 mm to (169.5, 30.1)
- moved C11 80.0 mm to (160.5, 33.0), turned to 0 degrees
- moved C2 79.6 mm to (162.1, 25.3)
- moved C13 75.7 mm to (171.3, 25.0), turned to 0 degrees
- moved C1 74.8 mm to (149.9, 34.5), turned to 0 degrees
- moved D2 71.2 mm to (155.3, 36.2), turned to 0 degrees
- moved P15 70.9 mm to (195.0, 25.5), turned to 0 degrees
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Connections:
- C1 pad 1: Earth -> 5V
- C1 pad 2: 3.3V -> Earth
- C11 pad 1: Earth -> Net-(C11-Pad1)
- C11 pad 2: 3.3V -> VCAP1
- C12 pad 1: Earth -> Net-(C11-Pad1)
- C12 pad 2: 3.3V -> VCAP1
- C13 pad 1: Earth -> Net-(C11-Pad1)
- C13 pad 2: 3.3V -> VCAP2
- C14 pad 1: 5V -> Net-(C11-Pad1)
- C14 pad 2: Earth -> VCAP2
- C15 pad 1: 3.3V -> NRST
- C2 pad 1: Earth -> 3.3V
- C2 pad 2: 3.3V -> Earth
- J1 pad 1: Earth -> BOOT
- J1 pad 2: Net-(J1-Pad2) -> Earth
- K1 pad 2: SOL1 -> Net-(K1-Pad2)
- K1 pad 4: Net-(K1-Pad4) -> Earth
- K2 pad 2: SOL2 -> Net-(K2-Pad2)
- K2 pad 4: Net-(K2-Pad4) -> Earth
- K3 pad 2: SOL3 -> Net-(K3-Pad2)
- K3 pad 4: Net-(K3-Pad4) -> Earth
- K4 pad 2: SOL5 -> Net-(K4-Pad2)
- K4 pad 4: Net-(K4-Pad4) -> Earth
- K5 pad 2: SOL6 -> Net-(K5-Pad2)
- K5 pad 4: Net-(K5-Pad4) -> Earth
- K6 pad 2: SOL4 -> Net-(K6-Pad2)
- K6 pad 4: Net-(K6-Pad4) -> Earth
- P1 pad 2: unconnected-(P1-Pad2) -> 3.3V
- P1 pad 3: unconnected-(P1-Pad3) -> Earth
- P1 pad 5: unconnected-(P1-Pad5) -> Earth
- R10 pad 1: Net-(K6-Pad4) -> SOL4
- R10 pad 2: Earth -> Net-(K6-Pad2)
- R2 pad 1: Net-(K1-Pad4) -> SOL1
- R2 pad 2: Earth -> Net-(K1-Pad2)
- R4 pad 1: Net-(K2-Pad4) -> SOL2
- R4 pad 2: Earth -> Net-(K2-Pad2)
- R5 pad 1: Net-(K3-Pad4) -> SOL3
- R5 pad 2: Earth -> Net-(K3-Pad2)
- R8 pad 1: Net-(K4-Pad4) -> SOL5
- R8 pad 2: Earth -> Net-(K4-Pad2)
- R9 pad 1: Net-(K5-Pad4) -> SOL6
- R9 pad 2: Earth -> Net-(K5-Pad2)
- U1 pad 1: unconnected-(U1-Pad1) -> SOL1
- U1 pad 10: unconnected-(U1-Pad10) -> Earth
- U1 pad 11: PG1 -> 3.3V
- U1 pad 12: PG2 -> unconnected-(U1-Pad12)
- U1 pad 13: VAC_MON -> unconnected-(U1-Pad13)
- U1 pad 14: unconnected-(U1-Pad14) -> NRST
- U1 pad 15: unconnected-(U1-Pad15) -> PG1
- U1 pad 16: unconnected-(U1-Pad16) -> PG2
- U1 pad 19: unconnected-(U1-Pad19) -> Earth
- U1 pad 2: unconnected-(U1-Pad2) -> SOL2
- U1 pad 20: Earth -> 3.3V
- U1 pad 21: Earth -> 3.3V
- U1 pad 22: 3.3V -> SOL4
- U1 pad 23: 3.3V -> SOL5
- U1 pad 24: 3.3V -> SOL6
- U1 pad 25: Earth -> unconnected-(U1-Pad25)
- U1 pad 26: unconnected-(U1-Pad26) -> Earth
- U1 pad 27: unconnected-(U1-Pad27) -> 3.3V
- U1 pad 3: unconnected-(U1-Pad3) -> SOL3
- U1 pad 31: RX -> unconnected-(U1-Pad31)
- U1 pad 32: TX -> unconnected-(U1-Pad32)
- U1 pad 33: Earth -> unconnected-(U1-Pad33)
- U1 pad 34: 3.3V -> unconnected-(U1-Pad34)
- U1 pad 36: SBV1_EN -> unconnected-(U1-Pad36)
- U1 pad 37: SBV1_DIR -> unconnected-(U1-Pad37)
- U1 pad 38: ENCD1_A -> unconnected-(U1-Pad38)
- U1 pad 39: SBV1_PUL -> unconnected-(U1-Pad39)
- U1 pad 4: unconnected-(U1-Pad4) -> SBV1_PUL
- U1 pad 40: ENCD1_B -> unconnected-(U1-Pad40)
- U1 pad 41: SBV2_PUL -> unconnected-(U1-Pad41)
- U1 pad 42: SBV2_EN -> unconnected-(U1-Pad42)
- U1 pad 43: SBV2_DIR -> unconnected-(U1-Pad43)
- U1 pad 45: ENCD2_A -> unconnected-(U1-Pad45)
- U1 pad 46: ENCD2_B -> unconnected-(U1-Pad46)
- U1 pad 47: SOL1 -> unconnected-(U1-Pad47)
- U1 pad 48: SOL2 -> VCAP1
- U1 pad 49: SOL3 -> Earth
- U1 pad 5: Net-(J1-Pad2) -> SBV2_PUL
- U1 pad 50: SWO -> 3.3V
- U1 pad 51: SOL5 -> unconnected-(U1-Pad51)
- U1 pad 52: SWCLK -> VAC_MON
- U1 pad 53: SWDIO -> unconnected-(U1-Pad53)
- U1 pad 54: SOL6 -> unconnected-(U1-Pad54)
- U1 pad 55: Earth -> unconnected-(U1-Pad55)
- U1 pad 56: 3.3V -> unconnected-(U1-Pad56)
- U1 pad 57: SOL4 -> unconnected-(U1-Pad57)
- U1 pad 6: Net-(J2-Pad2) -> unconnected-(U1-Pad6)
- U1 pad 62: EXECPT -> ENCD2_B
- U1 pad 63: STATUS -> ENCD2_A
- U1 pad 64: NRST -> SBV2_DIR
- U1 pad 8: 3.3V -> unconnected-(U1-Pad8)
- U1 pad 9: Earth -> unconnected-(U1-Pad9)
Routing:
- net Net-(K5-Pad2): track 0.00 -> 63.7 mm, vias 0 -> 3
- net SOL6: track 61.9 -> 0.00 mm, vias 2 -> 0
- net SOL5: track 56.3 -> 3.28 mm, vias 2 -> 0
- net Net-(K4-Pad2): track 0.00 -> 52.9 mm, vias 0 -> 3
- net Net-(K6-Pad2): track 0.00 -> 51.9 mm, vias 0 -> 3
- net SOL4: track 50.4 -> 0.00 mm, vias 2 -> 0
- net SOL3: track 34.3 -> 0.00 mm, vias 2 -> 0
- net Net-(K3-Pad2): track 0.00 -> 34.3 mm, vias 0 -> 2
- net Net-(K1-Pad2): track 0.00 -> 34.0 mm, vias 0 -> 1
- net VAC_MON: track 35.1 -> 2.25 mm, vias 2 -> 0
- net SOL1: track 32.7 -> 0.00 mm
- net 3.3V: track 92.2 -> 61.3 mm, vias 11 -> 5
- net SOL2: track 28.6 -> 0.00 mm
- net Earth: track 189.1 -> 171.4 mm, vias 24 -> 13
- net ENCD2_B: track 49.1 -> 31.5 mm, vias 2 -> 1
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